File: inker_super_board_ver0.sch (EAGLE design)
At the start: 31 parts, among them IC1 ATMEGA328P-AU, IC2 UA78L05AIPK, IC4 CH340G, J1 MC001667, J2 S2B-EH(LF)(SN), U1 NCP1117ST33T3G, Y1 MCRSD16000F183000RR., Y2 ABLS-12.000MHZ-B2-T

Commit message: Update inker_super_board_ver0.sch
Parts:
- added U2: ESP-32S, inker_super_board_parts:ESP-32S
Changed lines of the file:
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@@
 <part name="SUPPLY4" library="inker_blue_board_parts" deviceset="3.3V" device=""/>
 <part name="S2" library="inker_blue_board_parts" deviceset="1437566-3" device=""/>
+<part name="U2" library="inker_super_board_parts" deviceset="ESP-32S" device=""/>
 </parts>
 <sheets>
@@
 <attribute name="VALUE" x="78.74" y="78.232" size="1.778" layer="96" font="vector" align="top-center"/>
 </instance>
+<instance part="U2" gate="G$1" x="17.78" y="81.28" smashed="yes">
+<attribute name="NAME" x="52.07" y="88.9" size="1.778" layer="95" align="center-left"/>
+<attribute name="VALUE" x="52.07" y="86.36" size="1.778" layer="96" align="center-left"/>
+</instance>
 </instances>
